File: 8-bit-cpu-modules/ram.kicad_sch (KiCad schematic)
At the start: 0 parts

Commit message: Added some ram components
Parts:
- added D35, D36, D37, D38, D39, D40, D41, D42: LED, symbol Device:LED
- added R10, R11, R12, R13, R14, R7, R8, R9: 220, symbol Device:R
- added SW3: SW_DIP_x08, symbol Switch:SW_DIP_x08
- added U12, U13: 74LS157, symbol 74xx:74LS157
- added U14: 74HC245, symbol 74xx:74HC245
Connections:
- new net: D40.1 (K), R12.1
- new net: R11.2, R12.2, R13.2, R14.2
- new net: D38.1 (K), R10.1
- new net: D41.1 (K), R13.1
- new net: SW3.2, U13.11 (I0c)
- new net: SW3.1, U13.14 (I0d)
- new net: U12.15 (E), U12.8 (GND), U13.15 (E), U13.8 (GND)
- new net: SW3.4, U13.2 (I0a)
- new net: SW3.3, U13.5 (I0b)
- new net: R10.2, R7.2, R8.2, R9.2
- new net: D39.1 (K), R11.1
- new net: SW3.5, U12.14 (I0d)
- new net: SW3.6, U12.11 (I0c)
- new net: SW3.7, U12.5 (I0b)
- new net: SW3.8, U12.2 (I0a)
- new net: D37.1 (K), R9.1
- new net: D35.1 (K), R7.1
- new net: D36.1 (K), R8.1
- new net: D42.1 (K), R14.1
- new net BUS_0: U13.13 (I1d), U14.11 (B7)
- new net BUS_1: U13.10 (I1c), U14.12 (B6)
- new net BUS_2: U13.6 (I1b), U14.13 (B5)
- new net BUS_3: U13.3 (I1a), U14.14 (B4)
- new net BUS_4: U12.13 (I1d), U14.15 (B3)
- new net BUS_5: U12.10 (I1c), U14.16 (B2)
- new net BUS_6: U12.6 (I1b), U14.17 (B1)
- new net BUS_7: U12.3 (I1a), U14.18 (B0)
- new net PROG: U12.1 (S), U13.1 (S)
- new net ~{RO}: U14.19 (CE)
